File: start1.kicad_pcb (KiCad board)
At the start: 2 copper layers, 60 x 75 mm, 18 parts, among them Q1 MMBT3904, Q2 MMBT3904

Commit message: Wired it up! needs finishing touches
Parts:
- moved R4 13.5 mm to (38.5, 49.6), turned to 90 degrees
- moved R2 5.72 mm to (51.2, 49.7)
- moved R5 5.71 mm to (44.9, 49.7)
- moved R6 1.29 mm to (58.0, 40.0), turned to 180 degrees
- turned R1 to 0 degrees
- turned R3 to 270 degrees
Routing:
- net GND: track 237.0 -> 0.00 mm
- net VCC: track 181.4 -> 0.00 mm
- net Net-(C2-Pad1): track 142.9 -> 0.00 mm
- net Net-(C1-Pad2): track 62.2 -> 0.00 mm
- net Net-(C1-Pad1): track 60.2 -> 0.00 mm
- net Net-(C2-Pad2): track 54.1 -> 0.00 mm
- net Net-(D3-Pad1): track 10.8 -> 0.00 mm
- net Net-(D5-Pad1): track 7.46 -> 0.00 mm
- net Net-(D2-Pad1): track 7.46 -> 0.00 mm
- net Net-(D1-Pad1): track 7.46 -> 0.00 mm
- net Net-(D7-Pad1): track 3.47 -> 0.00 mm
- net Net-(D6-Pad1): track 2.46 -> 0.00 mm
- net Net-(D4-Pad1): track 2.46 -> 0.00 mm
Other:
- net class VCC removed
