File: working1.kicad_pcb (KiCad board)
At the start: 2 copper layers, 60 x 75 mm, 18 parts, among them Q1 MMBT3904, Q2 MMBT3904

Commit message: Wired it up! needs finishing touches
Parts:
- moved R6 1.29 mm to (58.0, 40.0), turned to 180 degrees
- turned R1 to 0 degrees
Routing:
- net GND: track 237.0 -> 192.1 mm
- net Net-(C2-Pad1): track 142.9 -> 132.0 mm
- net Net-(C2-Pad2): track 54.1 -> 46.1 mm
- net Net-(D7-Pad1): track 3.47 -> 10.5 mm
- net Net-(D3-Pad1): track 10.8 -> 15.7 mm
- net Net-(C1-Pad1): track 60.2 -> 57.0 mm
- net Net-(C1-Pad2): track 62.2 -> 62.7 mm
